File: PCB_Designs/MainBoard_PCB/Lab1.sch (KiCad schematic (older format))
At the start: 77 parts, among them K1 XLR3, P1 CONN_01X06, P2 USB_B, P3 CONN_02X05, P4 CONN_01X02, P5 CONN_02X05, Q1 BSS138, Q2 BSS138, Q3 BSS138, Q4 BSS138, Q5 BSS138, Q6 BSS138, Q7 BSS138, U1 STM32F411RETx, U10 24C16, U2 TRACO_POWER_DC/DC_CONVERTER, U3 6N137, U4 6N137, U5 6N137, U6 FT232RL, U7 MAX481CSA, U8 LM7805, U9 LM7833, Y1 8MHz

Commit message: PCB file created for main board
Nothing really
Parts:
- D1: symbol LED -> LED-RESCUE-Lab1
- P2: symbol USB_B -> USB_B-RESCUE-Lab1
Connections:
- no-connect marks 56 -> 60

Commit message: Main PCB work in progress...
Parts:
- removed U2: TRACO_POWER_DC/DC_CONVERTER, Housings_DIP:DIP-24_W7.62mm_Socket, symbol TRACO_POWER_DC/DC_CONVERTER
- removed U8: LM7805, TO_SOT_Packages_SMD:SOT-223-3Lead_TabPin2, symbol LM7805
- removed U9: LM7833, TO_SOT_Packages_SMD:SOT-223-3Lead_TabPin2, symbol LM7805
- added U2: DC/DC_CONV, Converters_DCDC_ACDC:DCDC-Conv_TRACO_TED-xxxx_Single, symbol DC/DC_CONV
- added U8: LT1129CST-5, TO_SOT_Packages_SMD:SOT-223, symbol LT1129CST-5
- added U9: LT1129CST-3.3, TO_SOT_Packages_SMD:SOT-223, symbol LT1129CST-3.3
- C12, C15, C18, C24: footprint Capacitors_SMD:CP_Elec_10x10.5 -> Capacitors_Tantalum_SMD:CP_Tantalum_Case-C_EIA-6032-28_Hand
- C13: value 100nC -> 100n
- U3, U4, U5: footprint DIP-8 -> Housings_DIP:DIP-8_W7.62mm_LongPads
Connections:
- net labels removed: VDD5
- wire segments 184 -> 180
Other:
- note removed: "NOTE: Pins are incorrect"
- moved on the sheet: C10, C14, C15, C20, C21, C22, C23, C24, C6, C7, C8, C9

Commit message: First PCB version of main board
Parts:
- added P6: CONN_02X05, Pin_Headers:Pin_Header_Straight_2x05_Pitch2.54mm, symbol CONN_02X05
- K1: footprint Connect:XLR3MC -> Pin_Headers:Pin_Header_Straight_1x03_Pitch1.27mm
Connections:
- wire segments 180 -> 187
- no-connect marks 60 -> 76
Changed lines of the file:
@@
 LIBS:contrib
 LIBS:valves
+LIBS:stm32
+LIBS:ft232rl
+LIBS:max3485e
+LIBS:DCDCconv
 LIBS:Lab1-cache
 EELAYER 25 0
@@
 NoConn ~ 3300 5550
 NoConn ~ 9100 2550
-NoConn ~ 9100 2850
-NoConn ~ 9100 3050
-NoConn ~ 9100 3150
 NoConn ~ 9100 3950
 NoConn ~ 9100 4250
@@
 NoConn ~ 9100 5350
 NoConn ~ 9100 5450
-NoConn ~ 9100 2950
 NoConn ~ 9100 4150
 NoConn ~ 9100 3650
@@
 F 0 "K1" H 7400 10200 50  0000 C CNN
 F 1 "XLR3" H 7450 9700 50  0000 C CNN
-F 2 "Connect:XLR3MC" H 7250 9950 50  0001 C CNN
+F 2 "Pin_Headers:Pin_Header_Straight_1x03_Pitch1.27mm" H 7250 9950 50  0001 C CNN
 F 3 "" H 7250 9950 50  0000 C CNN
 	1    7250 9950
@@
 Connection ~ 9350 700
 Connection ~ 9350 1450
+$Comp
+L CONN_02X05 P6
+U 1 1 58A11651
+P 10600 2950
+F 0 "P6" H 10600 3250 50  0000 C CNN
+F 1 "CONN_02X05" H 10600 2650 50  0000 C CNN
+F 2 "Pin_Headers:Pin_Header_Straight_2x05_Pitch2.54mm" H 10600 1750 50  0001 C CNN
+F 3 "" H 10600 1750 50  0000 C CNN
+	1    10600 2950
+	1    0    0    -1
+$EndComp
+$Comp
+L GND #PWR056
+U 1 1 58A11657
+P 10350 2850
+F 0 "#PWR056" H 10350 2600 50  0001 C CNN
+F 1 "GND" H 10350 2700 50  0000 C CNN
+F 2 "" H 10350 2850 50  0000 C CNN
+F 3 "" H 10350 2850 50  0000 C CNN
+	1    10350 2850
+	0    1    1    0
+$EndComp
+$Comp
+L +5V #PWR057
+U 1 1 58A1165D
+P 10350 2750
+F 0 "#PWR057" H 10350 2600 50  0001 C CNN
+F 1 "+5V" H 10350 2890 50  0000 C CNN
+F 2 "" H 10350 2750 50  0000 C CNN
+F 3 "" H 10350 2750 50  0000 C CNN
+	1    10350 2750
+	1    0    0    -1
+$EndComp
+NoConn ~ 10850 2850
+NoConn ~ 10850 2950
+NoConn ~ 10850 3050
+NoConn ~ 10850 3150
+Wire Wire Line
+	9100 3150 10350 3150
+Wire Wire Line
+	9100 3050 10350 3050
+Wire Wire Line
+	9100 2950 10350 2950
+Wire Wire Line
+	10850 2750 10850 2500
+Wire Wire Line
+	10850 2500 10100 2500
+Wire Wire Line
+	10100 2500 10100 2850
+Wire Wire Line
+	10100 2850 9100 2850
+NoConn ~ 2950 12300
+NoConn ~ 2950 12400
+NoConn ~ 2950 12500
+NoConn ~ 2950 12600
+NoConn ~ 2950 12700
+NoConn ~ 2950 12800
+NoConn ~ 2950 12900
+NoConn ~ 2950 13000
+NoConn ~ 4350 12300
+NoConn ~ 4350 12400
+NoConn ~ 4350 12500
+NoConn ~ 4350 12600
+NoConn ~ 4350 12700
+NoConn ~ 4350 12800
+NoConn ~ 4350 12900
+NoConn ~ 4350 13000
 $EndSCHEMATC

Commit message: Added 3.3v to FT232RL, use larger power tracks
Parts:
- U8: value LT1129CST-5 -> UA78M05IDCY
- U9: value LT1129CST-3.3 -> UA78M33CDCY
Connections:
- wire segments 187 -> 189
- no-connect marks 76 -> 75
Other:
- note added: "12V DC Jack"
- note added: "3.3V <-> 5V level conversion"
- note added: "Analog slide \npotentiometers\ninput"
- note added: "Backlight brightness\nthrough PWM"
- note added: "DMX512 output"
- note added: "Digital buttons\n(I/O Expander through I2C)"
- note added: "EEPROM"
- note added: "LCD and rotary encoder\n(I/O Expander through I2C)"
- note added: "Max 0.5A"
- note added: "SWD connector"
- moved on the sheet: R14, R9
Changed lines of the file:
@@
 LIBS:contrib
 LIBS:valves
-LIBS:stm32
 LIBS:ft232rl
 LIBS:max3485e
@@
 F 0 "U3" H 3600 9100 50  0000 L CNN
 F 1 "6N137" H 3800 9100 50  0000 L CNN
-F 2 "Housings_DIP:DIP-8_W7.62mm_LongPads" H 3600 8500 50  0000 L CIN
+F 2 "Housings_DIP:DIP-8_W7.62mm_LongPads" H 3050 8500 50  0000 L CIN
 F 3 "" H 3800 8800 50  0000 L CNN
 	1    3800 8800
-	-1   0    0    1
+	-1   0    0    -1
 $EndComp
 $Comp
@@
 F 0 "U4" H 3600 10150 50  0000 L CNN
 F 1 "6N137" H 3800 10150 50  0000 L CNN
-F 2 "Housings_DIP:DIP-8_W7.62mm_LongPads" H 3600 9550 50  0000 L CIN
+F 2 "Housings_DIP:DIP-8_W7.62mm_LongPads" H 3000 9550 50  0000 L CIN
 F 3 "" H 3800 9850 50  0000 L CNN
 	1    3800 9850
@@
 F 0 "U5" H 3600 11250 50  0000 L CNN
 F 1 "6N137" H 3800 11250 50  0000 L CNN
-F 2 "Housings_DIP:DIP-8_W7.62mm_LongPads" H 3600 10650 50  0000 L CIN
+F 2 "Housings_DIP:DIP-8_W7.62mm_LongPads" H 3100 10650 50  0000 L CIN
 F 3 "" H 3800 10950 50  0000 L CNN
 	1    3800 10950
@@
 L R R9
 U 1 1 589E0292
-P 2850 9000
-F 0 "R9" V 2930 9000 50  0000 C CNN
-F 1 "470" V 2850 9000 50  0000 C CNN
-F 2 "Resistors_SMD:R_0603_HandSoldering" V 2780 9000 50  0001 C CNN
-F 3 "" H 2850 9000 50  0000 C CNN
-	1    2850 9000
+P 3000 8600
+F 0 "R9" V 3080 8600 50  0000 C CNN
+F 1 "470" V 3000 8600 50  0000 C CNN
+F 2 "Resistors_SMD:R_0603_HandSoldering" V 2930 8600 50  0001 C CNN
+F 3 "" H 3000 8600 50  0000 C CNN
+	1    3000 8600
 	0    1    1    0
 $EndComp
@@
 L GND #PWR017
 U 1 1 589E03E9
-P 3200 8600
-F 0 "#PWR017" H 3200 8350 50  0001 C CNN
-F 1 "GND" H 3200 8450 50  0000 C CNN
-F 2 "" H 3200 8600 50  0000 C CNN
-F 3 "" H 3200 8600 50  0000 C CNN
-	1    3200 8600
-	-1   0    0    1
-$EndComp
-Text Label 4100 8900 0    60   ~ 0
+P 2900 9000
+F 0 "#PWR017" H 2900 8750 50  0001 C CNN
+F 1 "GND" H 2900 8850 50  0000 C CNN
+F 2 "" H 2900 9000 50  0000 C CNN
+F 3 "" H 2900 9000 50  0000 C CNN
+	1    2900 9000
+	1    0    0    -1
+$EndComp
+Text Label 4100 8700 0    60   ~ 0
 VDD5EXT
 $Comp
 L R R14
 U 1 1 589E056E
-P 4700 8700
-F 0 "R14" V 4780 8700 50  0000 C CNN
-F 1 "470" V 4700 8700 50  0000 C CNN
-F 2 "Resistors_SMD:R_0603_HandSoldering" V 4630 8700 50  0001 C CNN
-F 3 "" H 4700 8700 50  0000 C CNN
-	1    4700 8700
+P 4400 8900
+F 0 "R14" V 4480 8900 50  0000 C CNN
+F 1 "470" V 4400 8900 50  0000 C CNN
+F 2 "Resistors_SMD:R_0603_HandSoldering" V 4330 8900 50  0001 C CNN
+F 3 "" H 4400 8900 50  0000 C CNN
+	1    4400 8900
 	0    1    1    0
 $EndComp
@@
 $EndComp
 NoConn ~ 4100 9750
-NoConn ~ 3500 8900
+NoConn ~ 3500 8700
 $Comp
 L +5V #PWR018
@@
 	-1   0    0    1
 $EndComp
-NoConn ~ 3000 -2650
 NoConn ~ 3000 -1750
 NoConn ~ 3000 -1450
@@
 	1950 1450 1950 1050
 Wire Wire Line
-	3000 9000 3500 9000
-Wire Wire Line
-	3500 8700 2700 8700
-Wire Wire Line
-	3200 8600 3500 8600
-Wire Wire Line
-	4550 8700 4100 8700
-Wire Wire Line
-	4850 8700 4850 9950
-Wire Wire Line
 	4850 9950 5100 9950
 Wire Wire Line
@@
 Wire Wire Line
 	3100 9750 3100 9700
-Connection ~ 2700 9000
 Wire Wire Line
 	2400 9000 2400 9050
@@
 Wire Wire Line
 	2700 9450 2150 9450
-Connection ~ 2700 9450
-Wire Wire Line
-	2700 8700 2700 9450
 Wire Wire Line
 	1400 9450 1400 9350
@@
 P 8800 1500
 F 0 "U9" H 8550 1700 50  0000 C CNN
-F 1 "LT1129CST-3.3" H 8950 1700 50  0000 C CNN
+F 1 "UA78M33CDCY" H 8950 1700 50  0000 C CNN
 F 2 "TO_SOT_Packages_SMD:SOT-223" H 8800 1600 50  0000 C CIN
 F 3 "" H 8800 1500 50  0000 C CNN
@@
 P 8800 750
 F 0 "U8" H 8550 950 50  0000 C CNN
-F 1 "LT1129CST-5" H 8950 950 50  0000 C CNN
+F 1 "UA78M05IDCY" H 8950 950 50  0000 C CNN
 F 2 "TO_SOT_Packages_SMD:SOT-223" H 8800 850 50  0000 C CIN
 F 3 "" H 8800 750 50  0000 C CNN
@@
 NoConn ~ 4350 12900
 NoConn ~ 4350 13000
+$Comp
+L +3V3 #PWR058
+U 1 1 58A512E3
+P 3000 -2650
+F 0 "#PWR058" H 3000 -2800 50  0001 C CNN
+F 1 "+3V3" H 3000 -2510 50  0000 C CNN
+F 2 "" H 3000 -2650 50  0000 C CNN
+F 3 "" H 3000 -2650 50  0000 C CNN
+	1    3000 -2650
+	1    0    0    -1
+$EndComp
+Text Notes 10350 3600 0    60   ~ 0
+Analog slide \npotentiometers\ninput
+Text Notes 10600 5700 0    60   ~ 0
+EEPROM
+Text Notes 10900 9500 0    60   ~ 0
+LCD and rotary encoder\n(I/O Expander through I2C)
+Text Notes 6900 10450 0    60   ~ 0
+DMX512 output
+Text Notes 2350 7400 0    60   ~ 0
+Digital buttons\n(I/O Expander through I2C)
+Text Notes 6300 1000 0    60   ~ 0
+12V DC Jack
+Wire Wire Line
+	4550 8900 4850 8900
+Wire Wire Line
+	4850 8900 4850 9950
+Wire Wire Line
+	4250 8900 4100 8900
+Wire Wire Line
+	3500 9000 2900 9000
+Wire Wire Line
+	3150 8600 3500 8600
+Wire Wire Line
+	2700 8600 2850 8600
+Wire Wire Line
+	2700 8600 2700 9450
+Wire Wire Line
+	3500 8900 2700 8900
+Connection ~ 2700 8900
+$Comp
+L +5V #PWR059
+U 1 1 58A8BFF0
+P 3300 8600
+F 0 "#PWR059" H 3300 8450 50  0001 C CNN
+F 1 "+5V" H 3300 8740 50  0000 C CNN
+F 2 "" H 3300 8600 50  0000 C CNN
+F 3 "" H 3300 8600 50  0000 C CNN
+	1    3300 8600
+	1    0    0    -1
+$EndComp
+Text Notes 9900 1350 0    60   ~ 0
+Max 0.5A
+Text Notes 9850 600  0    60   ~ 0
+Max 0.5A
+Text Notes 8150 12250 0    60   ~ 0
+Backlight brightness\nthrough PWM
+Wire Notes Line
+	2550 11750 2550 8600
+Wire Notes Line
+	2550 8600 450  8600
+Wire Notes Line
+	450  8600 450  11750
+Wire Notes Line
+	450  11750 2550 11750
+Text Notes 450  11900 0    60   ~ 0
+3.3V <-> 5V level conversion
+Wire Notes Line
+	10600 12500 10600 8450
+Wire Notes Line
+	10600 8450 7950 8450
+Wire Notes Line
+	7950 8450 7950 12500
+Wire Notes Line
+	7950 12500 10600 12500
+Text Notes 7950 12650 0    60   ~ 0
+3.3V <-> 5V level conversion
+Text Notes 1100 1950 0    60   ~ 0
+SWD connector
 $EndSCHEMATC

Commit message: Fixed DC DC converter footprint
Parts:
- removed U2: DC/DC_CONV, Converters_DCDC_ACDC:DCDC-Conv_TRACO_TED-xxxx_Single, symbol DC/DC_CONV
- added U2: TRACO_POWER_TEL_2-0511, symbol TRACO_POWER_TEL_2-0511
Connections:
- no-connect marks 75 -> 71
Other:
- note added: "DC/DC converter"
- note removed: "3.3V <-> 5V level conversion"
- note removed: "SWD connector"
- moved on the sheet: C20, C21, C22

Commit message: Rerouted MCU pins for better Nucleo compatibility
Parts:
- U2: footprint (none) -> LIBRARIES:TRACO_POWER_TEX_2-0511
Connections:
- net +5V: now also P6.2 (P2); no longer P6.1 (P1)
- net GND: now also P6.1 (P1); no longer P6.3 (P3)
- net INT_ROTARY: now also U1.26 (ADC1_IN8/I2S5_CK/SPI5_SCK/TIM1_CH2N/TIM3_CH3/PB0); no longer U1.58 (I2C1_SCL/TIM4_CH1/USART1_TX/PB6)
- net LCD_I2C_SCL: now also U1.58 (I2C1_SCL/TIM4_CH1/USART1_TX/PB6); no longer U1.29 (I2C2_SCL/I2S2_CK/I2S3_MCK/SDIO_D7/SPI2_SCK/TIM2_CH3/PB10)
- net LCD_I2C_SDA: now also U1.59 (I2C1_SDA/SDIO_D0/TIM4_CH2/USART1_RX/PB7); no longer U1.55 (I2C2_SDA/I2S1_CK/I2S3_CK/SPI1_SCK/SPI3_SCK/SYS_JTDO-SWO/TIM2_CH2/USART1_RX/PB3)
- net at U1.10 (PC2/ADC1_IN12/I2S2_ext_SD/SPI2_MISO): now also P6.7 (P7)
- net at U1.11 (PC3/ADC1_IN13/I2S2_SD/SPI2_MOSI): now also P6.9 (P9)
- net at U1.20 (ADC1_IN4/I2S1_WS/I2S3_WS/SPI1_NSS/SPI3_NSS/USART2_CK/PA4): no longer P6.2 (P2)
- net at U1.21 (ADC1_IN5/I2S1_CK/SPI1_SCK/TIM2_CH1/TIM2_ETR/PA5): no longer P6.5 (P5)
- net at U1.22 (ADC1_IN6/I2S2_MCK/SDIO_CMD/SPI1_MISO/TIM1_BKIN/TIM3_CH1/PA6): no longer P6.7 (P7)
- net at U1.23 (ADC1_IN7/I2S1_SD/SPI1_MOSI/TIM1_CH1N/TIM3_CH2/PA7): no longer P6.9 (P9)
- net at U1.61 (I2C1_SCL/I2C3_SDA/I2S5_SD/SDIO_D4/SPI5_MOSI/TIM10_CH1/TIM4_CH3/PB8): no longer U10.6 (SCL)
- net EEPROM_I2C_SDA: now reaches U1.62 (I2C1_SDA/I2C2_SDA/I2S2_WS/SDIO_D5/SPI2_NSS/TIM11_CH1/TIM4_CH4/PB9), U10.5 (SDA)
- net at U1.8 (PC0/ADC1_IN10): now also P6.3 (P3)
- net at U1.9 (PC1/ADC1_IN11): now also P6.5 (P5)
- new net EEPROM_I2C_SCL: U1.29 (I2C2_SCL/I2S2_CK/I2S3_MCK/SDIO_D7/SPI2_SCK/TIM2_CH3/PB10), U10.6 (SCL)
Other:
- moved on the sheet: P6, U10

Commit message: Main_PCB V1 Complete
Minor changes to everything.
Main_PCB complete with traces and design.
Parts:
- removed C4: 100n, Capacitors_SMD:C_0603_HandSoldering, symbol C
- removed C5, C6: 4.7u, Capacitors_SMD:C_0603_HandSoldering, symbol C
- added C4, C5, C6: 4.7u, Capacitors_Tantalum_SMD:CP_Tantalum_Case-A_EIA-3216-18_Reflow, symbol CP
- added P10, P11, P12, P7, P8, P9: CONN_01X01, Mounting_Holes:MountingHole_2.2mm_M2_DIN965_Pad, symbol CONN_01X01
- C12, C15, C18, C24: footprint Capacitors_Tantalum_SMD:CP_Tantalum_Case-C_EIA-6032-28_Hand -> Capacitors_Tantalum_SMD:CP_Tantalum_Case-A_EIA-3216-18_Reflow
- D1: footprint LEDs:LED_0603 -> LEDs:LED_D5.0mm
- D2: footprint Diodes_SMD:D_0603 -> Diodes_SMD:D_SOD-123
- L1: footprint Resistors_SMD:R_0603 -> Resistors_SMD:R_1206_HandSoldering
- P3, P5, P6: footprint Pin_Headers:Pin_Header_Straight_2x05_Pitch2.54mm -> Connectors_Multicomp:Multicomp_MC9A22-1034_2x05x2.54mm_Angled
- Y1: footprint Crystals:Crystal_SMD_HC49-SD_HandSoldering -> Crystals:Crystal_SMD_HC49-SD
Connections:
- net +12V: now also D2.2 (A), P4.2 (P2); no longer C11.1, C12.1, C13.1, D2.1 (K), U8.1 (VIN), U9.1 (VIN)
- net +3V3: now also P3.2 (P2), C4.1, C6.1
- net +5V: now also R9.1, U3.8
- net BUTT_I2C_SCL: now also P3.8 (P8)
- net BUTT_I2C_SDA: now also P3.6 (P6)
- net GND: now also C21.2, P3.4 (P4), P5.4 (P4), C4.2, C5.2, C6.2
- net GNDEXT: no longer C21.2
- net INT_BUTTA: now also P3.10 (P10)
- net VDD5EXT: no longer C21.1
- net at U1.10 (PC2/ADC1_IN12/I2S2_ext_SD/SPI2_MISO): now also P6.5 (P5), P6.6 (P6); no longer P6.7 (P7)
- net at U1.11 (PC3/ADC1_IN13/I2S2_SD/SPI2_MOSI): now also P6.3 (P3), P6.4 (P4); no longer P6.9 (P9)
- net at U1.30 (VCAP1): now also C5.1
- net at U1.8 (PC0/ADC1_IN10): now also P6.10 (P10), P6.9 (P9); no longer P6.3 (P3)
- net at U1.9 (PC1/ADC1_IN11): now also P6.7 (P7), P6.8 (P8); no longer P6.5 (P5)
- net at P5.5 (P5), Q7.3 (D), R26.1: now also P5.6 (P6)
- net at P5.7 (P7), Q4.3 (D), R23.1: now also P5.8 (P8)
- net at P5.9 (P9), Q5.3 (D), R24.1: now also P5.10 (P10)
- net INT_BUTTB: no longer names the net of U1.39 (PC8/SDIO_D0/TIM3_CH3/USART6_CK)
- net INT_BUTTB: no longer P3.2 (P2)
- new net: C11.1, C12.1, C13.1, C21.1, D2.1 (K), U8.1 (VIN), U9.1 (VIN)
- no-connect marks 71 -> 56
Other:
- note added: "Mounting\nHoles"
- moved on the sheet: C11, C12, C13, C22, D1, D2, P4, R18
