File: PCB_Designs/MainBoard_PCB/Lab1.sch (KiCad schematic (older format))
At the start: 92 parts, among them K1 XLR3, P1 CONN_01X06, P10 CONN_01X01, P11 CONN_01X01, P12 CONN_01X01, P2 USB_B, P3 CONN_02X05, P4 CONN_01X02, P5 CONN_02X05, P6 CONN_02X05, P7 CONN_01X01, P8 CONN_01X01, P9 CONN_01X01, Q1 BSS138, Q2 BSS138, Q3 BSS138, Q4 BSS138, Q5 BSS138, Q6 BSS138, Q7 BSS138, U1 STM32F411RETx, U10 24C16, U2 TRACO_POWER_TEL_2-0511, U3 6N137, U4 6N137, U5 6N137, U6 FT232RL, U7 MAX481CSA, U8 UA78M05IDCY, U9 UA78M33CDCY, Y1 8MHz

Commit message: Added pullups for EEPROM and button I/Os
Parts:
- added R31, R32, R33, R34: 10K, Resistors_SMD:R_0603_HandSoldering, symbol R
Connections:
- net +3V3: now also R31.2, R32.2, R33.2, R34.2
- net BUTT_I2C_SCL: now also R31.1
- net BUTT_I2C_SDA: now also R32.1
- net EEPROM_I2C_SCL: now also R33.1
- net EEPROM_I2C_SDA: now also R34.1
- net GND: now also U10.1 (A0)
- no-connect marks 56 -> 55
