File: PCB_Designs/OLED_LCD/OLED_LCD.sch (KiCad schematic (older format))
At the start: 28 parts, among them P1 CONN_01X10, P2 CONN_01X16, P3 CONN_01X01, P4 CONN_01X01, P5 CONN_01X01, P6 CONN_01X01, SW1 Rotary_Encoder_Switch, U1 MCP23017, U2 MCP23017, U3 CHERRY-MX

Commit message: Hej
Parts:
- removed U1: MCP23017, Housings_SOIC:SOIC-28W_7.5x17.9mm_Pitch1.27mm, symbol MCP23017
Connections:
- net BUTTON_2: now also U2.22 (GPA1)
- net BUTT_LED: now also U2.21 (GPA0)
- net E: now also U2.28 (GPA7); no longer U2.25 (GPA4)
- net ENCODERA: now also U2.25 (GPA4)
- net ENCODERB: now also U2.24 (GPA3)
- net ENCODERSW: now also U2.23 (GPA2)
- net INTA: now also U2.20 (INTA)
- net RS: now also U2.26 (GPA5); no longer U2.23 (GPA2)
- net RW: now also U2.27 (GPA6); no longer U2.24 (GPA3)
- net VCC5: now also U2.18 (~RESET)
- no-connect marks 25 -> 6
Changed lines of the file:
@@
 Comment4 ""
 $EndDescr
-$Comp
-L MCP23017 U2
-U 1 1 5894F8CE
-P 4550 3350
-F 0 "U2" H 4450 4375 50  0000 R CNN
-F 1 "MCP23017" H 4450 4300 50  0000 R CNN
-F 2 "Housings_SOIC:SOIC-28W_7.5x17.9mm_Pitch1.27mm" H 4600 2400 50  0001 L CNN
-F 3 "" H 4800 4350 50  0001 C CNN
-	1    4550 3350
-	1    0    0    -1
-$EndComp
 Text Label 4050 2550 2    60   ~ 0
 D0
@@
 Connection ~ 5150 4150
 $Comp
-L GND #PWR3
+L GND #PWR01
 U 1 1 5894FC28
 P 5150 4300
-F 0 "#PWR3" H 5150 4050 50  0001 C CNN
+F 0 "#PWR01" H 5150 4050 50  0001 C CNN
 F 1 "GND" H 5150 4150 50  0000 C CNN
 F 2 "" H 5150 4300 50  0000 C CNN
@@
 $EndComp
 $Comp
-L GND #PWR5
+L GND #PWR02
 U 1 1 5894FCE6
 P 6300 3250
-F 0 "#PWR5" H 6300 3000 50  0001 C CNN
+F 0 "#PWR02" H 6300 3000 50  0001 C CNN
 F 1 "GND" H 6300 3100 50  0000 C CNN
 F 2 "" H 6300 3250 50  0000 C CNN
@@
 Text Label 5050 3750 0    60   ~ 0
 SDA#
-Text Label 4050 3650 2    60   ~ 0
+Text Label 4050 3950 2    60   ~ 0
 RS
-Text Label 4050 3750 2    60   ~ 0
+Text Label 4050 4050 2    60   ~ 0
 RW
-Text Label 4050 3850 2    60   ~ 0
+Text Label 4050 4150 2    60   ~ 0
 E
 Text Label 7300 2300 2    60   ~ 0
@@
 LED-
 $Comp
-L GND #PWR7
+L GND #PWR03
 U 1 1 589508C9
 P 6600 4350
-F 0 "#PWR7" H 6600 4100 50  0001 C CNN
+F 0 "#PWR03" H 6600 4100 50  0001 C CNN
 F 1 "GND" H 6600 4200 50  0000 C CNN
 F 2 "" H 6600 4350 50  0000 C CNN
@@
 GND
 $Comp
-L GND #PWR9
+L GND #PWR04
 U 1 1 58950905
 P 7100 3900
-F 0 "#PWR9" H 7100 3650 50  0001 C CNN
+F 0 "#PWR04" H 7100 3650 50  0001 C CNN
 F 1 "GND" H 7100 3750 50  0000 C CNN
 F 2 "" H 7100 3900 50  0000 C CNN
@@
 	1    0    0    -1
 $EndComp
-$Comp
-L MCP23017 U1
-U 1 1 58950F84
-P 2000 3350
-F 0 "U1" H 1900 4375 50  0000 R CNN
-F 1 "MCP23017" H 1900 4300 50  0000 R CNN
-F 2 "Housings_SOIC:SOIC-28W_7.5x17.9mm_Pitch1.27mm" H 2050 2400 50  0001 L CNN
-F 3 "" H 2250 4350 50  0001 C CNN
-	1    2000 3350
-	1    0    0    -1
-$EndComp
-Wire Wire Line
-	2500 4050 2500 4350
-$Comp
-L GND #PWR1
-U 1 1 58951194
-P 2500 4350
-F 0 "#PWR1" H 2500 4100 50  0001 C CNN
-F 1 "GND" H 2500 4200 50  0000 C CNN
-F 2 "" H 2500 4350 50  0000 C CNN
-F 3 "" H 2500 4350 50  0000 C CNN
-	1    2500 4350
-	1    0    0    -1
-$EndComp
-Connection ~ 2500 4150
-Text Label 2500 3650 0    60   ~ 0
-SCL#
-Text Label 2500 3750 0    60   ~ 0
-SDA#
-Text Label 2500 3050 0    60   ~ 0
+Text Label 5050 3050 0    60   ~ 0
 INTA
-Text Label 2000 4350 0    60   ~ 0
-GND
-Text Label 1500 3450 2    60   ~ 0
+Text Label 4050 3850 2    60   ~ 0
 ENCODERA
-Text Label 1500 3550 2    60   ~ 0
+Text Label 4050 3750 2    60   ~ 0
 ENCODERB
-Text Label 1500 3650 2    60   ~ 0
+Text Label 4050 3650 2    60   ~ 0
 ENCODERSW
 $Comp
@@
 Connection ~ 4050 3750
 Connection ~ 4050 3850
-NoConn ~ 4050 4050
-NoConn ~ 4050 4150
 NoConn ~ 5050 2950
-NoConn ~ 5050 3050
-NoConn ~ 1500 2550
-NoConn ~ 1500 2650
-NoConn ~ 1500 2750
-NoConn ~ 1500 2850
-NoConn ~ 1500 2950
-NoConn ~ 1500 3050
-NoConn ~ 1500 3150
-NoConn ~ 1500 3250
 $Comp
 L CONN_01X10 P1
@@
 Wire Wire Line
 	5050 3750 5500 3750
-Connection ~ 2000 2350
-NoConn ~ 1500 3950
-NoConn ~ 1500 4050
-NoConn ~ 1500 4150
-Connection ~ 2500 3050
 Text Label 5800 1650 2    60   ~ 0
 INTA
@@
 Connection ~ 4300 1750
 $Comp
-L GND #PWR2
+L GND #PWR05
 U 1 1 58A0D2DB
 P 4300 2050
-F 0 "#PWR2" H 4300 1800 50  0001 C CNN
+F 0 "#PWR05" H 4300 1800 50  0001 C CNN
 F 1 "GND" H 4300 1900 50  0000 C CNN
 F 2 "" H 4300 2050 50  0000 C CNN
@@
 	1    0    0    -1
 $EndComp
-Text Label 1500 3750 2    60   ~ 0
+Text Label 4050 3550 2    60   ~ 0
 BUTTON_2
 Text Label 8000 1050 0    60   ~ 0
 BUTTON_2
 $Comp
-L GND #PWR8
+L GND #PWR06
 U 1 1 58A0E8E0
 P 6950 1650
-F 0 "#PWR8" H 6950 1400 50  0001 C CNN
+F 0 "#PWR06" H 6950 1400 50  0001 C CNN
 F 1 "GND" H 6950 1500 50  0000 C CNN
 F 2 "" H 6950 1650 50  0000 C CNN
@@
 	0    1    1    0
 $EndComp
-Text Label 1500 3850 2    60   ~ 0
+Text Label 4050 3450 2    60   ~ 0
 BUTT_LED
 Text Label 7550 1650 0    60   ~ 0
@@
 $EndComp
 $Comp
-L GND #PWR4
+L GND #PWR07
 U 1 1 58A0F70D
 P 5800 1050
-F 0 "#PWR4" H 5800 800 50  0001 C CNN
+F 0 "#PWR07" H 5800 800 50  0001 C CNN
 F 1 "GND" H 5800 900 50  0000 C CNN
 F 2 "" H 5800 1050 50  0000 C CNN
@@
 Text Label 5800 3750 0    60   ~ 0
 VCC5
-Text Label 2500 3950 0    60   ~ 0
-VCC5
 Text Label 4550 2350 0    60   ~ 0
-VCC5
-Text Label 2000 2350 0    60   ~ 0
 VCC5
 $Comp
@@
 VCC5
 $Comp
-L GND #PWR6
+L GND #PWR08
 U 1 1 58A10FD4
 P 6500 1050
-F 0 "#PWR6" H 6500 800 50  0001 C CNN
+F 0 "#PWR08" H 6500 800 50  0001 C CNN
 F 1 "GND" H 6500 900 50  0000 C CNN
 F 2 "" H 6500 1050 50  0000 C CNN
@@
 $EndComp
 $Comp
-L GND #PWR10
+L GND #PWR09
 U 1 1 58A1101A
 P 7550 1350
-F 0 "#PWR10" H 7550 1100 50  0001 C CNN
+F 0 "#PWR09" H 7550 1100 50  0001 C CNN
 F 1 "GND" H 7550 1200 50  0000 C CNN
 F 2 "" H 7550 1350 50  0000 C CNN
@@
 Text Label 7300 3700 2    60   ~ 0
 LCD_BACKLIGHT
-NoConn ~ 5050 2550
-NoConn ~ 2500 2950
 Wire Wire Line
 	5800 1050 5800 1150
@@
 	1    0    0    -1
 $EndComp
-NoConn ~ 4050 3450
-NoConn ~ 4050 3550
-NoConn ~ 4050 3950
-Text Label 2500 2550 0    60   ~ 0
-VCC5
-$Comp
-L PWR_FLAG #FLG1
+$Comp
+L PWR_FLAG #FLG010
 U 1 1 58B2ED0B
 P 6300 2800
-F 0 "#FLG1" H 6300 2875 50  0001 C CNN
+F 0 "#FLG010" H 6300 2875 50  0001 C CNN
 F 1 "PWR_FLAG" H 6300 2950 50  0000 C CNN
 F 2 "" H 6300 2800 50  0001 C CNN
@@
 $EndComp
 $Comp
-L PWR_FLAG #FLG2
+L PWR_FLAG #FLG011
 U 1 1 58B2EF20
 P 6300 3100
-F 0 "#FLG2" H 6300 3175 50  0001 C CNN
+F 0 "#FLG011" H 6300 3175 50  0001 C CNN
 F 1 "PWR_FLAG" H 6300 3250 50  0000 C CNN
 F 2 "" H 6300 3100 50  0001 C CNN
@@
 	0    1    1    0
 $EndComp
+Text Label 5050 2550 0    60   ~ 0
+VCC5
+$Comp
+L MCP23017 U2
+U 1 1 5894F8CE
+P 4550 3350
+F 0 "U2" H 4450 4375 50  0000 R CNN
+F 1 "MCP23017" H 4450 4300 50  0000 R CNN
+F 2 "Housings_SOIC:SOIC-28W_7.5x17.9mm_Pitch1.27mm" H 4600 2400 50  0001 L CNN
+F 3 "" H 4800 4350 50  0001 C CNN
+	1    4550 3350
+	1    0    0    -1
+$EndComp
 $EndSCHEMATC

Commit message: New stuff
Connections:
- net at 10k3.1, 10k4.2: now also SW1.3 (B); no longer SW1.1 (A)
- net at 10k1.2, 10k2.2: now also SW1.1 (A); no longer SW1.3 (B)
Changed lines of the file:
@@
 	1    0    0    -1
 $EndComp
-Text Label 3700 1100 2    60   ~ 0
+Text Label 3700 1100 0    60   ~ 0
 ENCODERA
 Text Label 2500 1100 2    60   ~ 0
@@
 	2500 1100 2700 1100
 Wire Wire Line
-	2400 1750 2400 1950
-Wire Wire Line
-	2400 1950 3400 1950
+	2400 1750 2400 1900
 Text Label 3400 1850 2    60   ~ 0
 GND
@@
 GND
 Connection ~ 3100 1750
-Connection ~ 3350 1750
-Connection ~ 2700 1950
+Connection ~ 2700 1900
 Text Label 3300 800  1    60   ~ 0
 GND
@@
 Connection ~ 3300 1750
 Wire Wire Line
-	2700 1550 2700 1950
+	2700 1550 2700 1900
 Wire Wire Line
 	3300 1100 3300 1250
@@
 Text Label 5800 1650 2    60   ~ 0
 INTA
-Wire Wire Line
-	3100 1750 3400 1750
 $Comp
 L C 100n4
@@
 	1    0    0    -1
 $EndComp
+Wire Wire Line
+	3300 1750 3100 1750
+Wire Wire Line
+	3100 1750 3100 1950
+Wire Wire Line
+	3100 1950 3400 1950
+Wire Wire Line
+	3400 1750 3350 1750
+Wire Wire Line
+	3350 1900 3350 1750
+Wire Wire Line
+	2400 1900 3350 1900
 $EndSCHEMATC
